File: KiCAD/MainBoard/MainBoard.kicad_sch (KiCad schematic)
At the start: 74 parts, among them J1 DB25, J2 Raspberry_Pi_2_3, P10 CONN_01X03, P11 CONN_01X03, P12 CONN_01X03, P13 CONN_01X03, P14 CONN_01X02, P15 CONN_02X07, P16 CONN_02X04, P18 CONN_01X03, P2 CONN_01X04, P3 CONN_02X04, P4 HOLE, P5 HOLE, P6 HOLE, P7 HOLE, P8 CONN_01X02, P9 CONN_01X03, Q1 BSS138, Q2 BSS138, Q3 DMN65D8L, U1 mp2307, U10 SI4425DDY, U11 INA199A2, U12 ADS1015, U2 DYS_mini_ESC, U3 DYS_mini_ESC, U4 DYS_mini_ESC, U5 DYS_mini_ESC, U6 TLV1117LV33, U7 TENDA_P200, U8 pca9685

Commit message: clean up the home plug and other things not on grid
Parts:
- C1, C19, C20, C22, C6, C7, C8, C9: symbol MainBoard-rescue:CP1 -> Device:C_Polarized_Small
- C10, C11, C12, C2, C21, C23, C24, C3, C4, C5: symbol MainBoard-rescue:C -> Device:C_Small
Connections:
- net GND: now also U1.4 (GND), U1.9 (GND)
- net V_BAT: now also U1.2 (IN)
- net at U1.1 (BS): now also C4.2
- net at U1.6 (COMP): now also C3.1
- no-connect marks 12 -> 11
Other:
- moved on the sheet: D1, D2, R6, R7, U1

Commit message: BLDC controller clean up
Parts:
- added C13, C14, C15, C16: 220uF/25V, Capacitor_SMD:CP_Elec_8x10, symbol Device:C_Polarized_Small
- added P1: CONN_02X04, Socket_Strips:Socket_Strip_Straight_2x04, symbol MainBoard-rescue:CONN_02X04
- added RN4: 20k, Resistors_SMD:R_Array_Concave_4x0603, symbol MainBoard-rescue:R_Pack04
- added U13, U14, U15, U9: DYS_mini_ESC, footprint:DYS_Mini_ESC, symbol custom_lib:DYS_mini_ESC
- C6, C7, C8, C9: footprint Capacitors_SMD:CP_Elec_8x10 -> Capacitor_SMD:CP_Elec_8x10
Connections:
- net GND: now also C13.2, C14.2, C15.2, C16.2, U13.1 (GND), U14.1 (GND), U15.1 (GND), U9.1 (GND)
- net V_PWR: now also C13.1, C14.1, C15.1, C16.1, U13.3 (VCC), U14.3 (VCC), U15.3 (VCC), U9.3 (VCC)
- net at U8.19 (PWM12): now also RN4.1 (R1.1)
- net at U8.20 (PWM13): now also RN4.2 (R2.1)
- net at U8.21 (PWM14): now also RN4.3 (R3.1)
- net at U8.22 (PWM15): now also RN4.4 (R4.1)
- new net CH12: P1.2 (P2), RN4.8 (R1.2)
- new net CH13: P1.4 (P4), RN4.7 (R2.2)
- new net CH14: P1.6 (P6), RN4.6 (R3.2)
- new net CH15: P1.8 (P8), RN4.5 (R4.2)
- new net ESC5: P1.1 (P1), U9.2 (PWM)
- new net ESC6: P1.3 (P3), U13.2 (PWM)
- new net ESC7: P1.5 (P5), U14.2 (PWM)
- new net ESC8: P1.7 (P7), U15.2 (PWM)
- new net MOTOR_5A: U9.4 (OUT_A)
- new net MOTOR_5B: U9.5 (OUT_B)
- new net MOTOR_5C: U9.6 (OUT_C)
- new net MOTOR_6A: U13.4 (OUT_A)
- new net MOTOR_6B: U13.5 (OUT_B)
- new net MOTOR_6C: U13.6 (OUT_C)
- new net MOTOR_7A: U14.4 (OUT_A)
- new net MOTOR_7B: U14.5 (OUT_B)
- new net MOTOR_7C: U14.6 (OUT_C)
- new net MOTOR_8A: U15.4 (OUT_A)
- new net MOTOR_8B: U15.5 (OUT_B)
- new net MOTOR_8C: U15.6 (OUT_C)
- no-connect marks 11 -> 7
Other:
- note added: "BLDC ESC X 8"
- note removed: "BLDC ESC X 4"
- moved on the sheet: C12, C6, C7, C8, C9, D1, D2, P14, P3, Q3, R15, R16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
