File: KiCAD/MainBoard/MainBoard.kicad_sch (KiCad schematic)
At the start: 84 parts, among them J1 DB25, J2 Raspberry_Pi_2_3, P1 CONN_02X04, P10 CONN_01X03, P11 CONN_01X03, P12 CONN_01X03, P13 CONN_01X03, P14 CONN_01X02, P15 CONN_02X07, P16 CONN_02X04, P18 CONN_01X03, P2 CONN_01X04, P3 CONN_02X04, P4 HOLE, P5 HOLE, P6 HOLE, P7 HOLE, P8 CONN_01X02, P9 CONN_01X03, Q1 BSS138, Q2 BSS138, Q3 DMN65D8L, U1 mp2307, U10 SI4425DDY, U11 INA199A2, U12 ADS1015, U13 DYS_mini_ESC, U14 DYS_mini_ESC, U15 DYS_mini_ESC, U2 DYS_mini_ESC, U3 DYS_mini_ESC, U4 DYS_mini_ESC, U5 DYS_mini_ESC, U6 TLV1117LV33, U7 TENDA_P200, U8 pca9685, U9 DYS_mini_ESC

Commit message: Update MainBoard.kicad_sch
Connections:
- net V_PWR renamed +V_PWR
