File: KiCAD/LED Lights/ledCube.kicad_pcb (KiCad board)
At the start: 2 copper layers, 52 x 22 mm, 14 parts, among them P1 Power, P2 LED +VE, P3 LED -VE, P4 LED +VE, P5 LED -VE, U1 AL8805W5

Commit message: update pcb
Parts:
- U1: value AL8805W5 -> AL8860WT-7
Routing:
- added copper zone on B.Cu, net /LED+/U
- added copper zone on B.Cu, net /LED-/U
Changed lines of the file:
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@@
+			)
+		)
+		(property "Vendor" "DigiKey"
+			(at 0 0 0)
+			(unlocked yes)
+			(layer "F.Fab")
+			(hide yes)
+			(effects
+				(font
+					(size 1 1)
+					(thickness 0.15)
+				)
 			)
 		)
@@
 			)
 		)
+		(property "Vendor" "DigiKey"
+			(at 0 0 270)
+			(unlocked yes)
+			(layer "F.Fab")
+			(hide yes)
+			(effects
+				(font
+					(size 1 1)
+					(thickness 0.15)
+				)
+			)
+		)
 		(property ki_fp_filters "Choke_* *Coil* Inductor_* L_*")
 		(sheetname "/")
@@
 			)
 		)
-		(property "Value" "AL8805W5"
+		(property "Value" "AL8860WT-7"
 			(at 0 2.9 180)
 			(layer "F.Fab")
@@
 			)
 		)
-		(property "Datasheet" "https://cdn.sparkfun.com/datasheets/Components/LED/AL8805.pdf"
+		(property "Datasheet" "https://www.diodes.com/assets/Datasheets/AL8860.pdf"
 			(at 0 0 180)
 			(layer "F.Fab")
@@
 			)
 		)
-		(property "Part #" "AL8805W5-7DICT-ND"
+		(property "Part #" "AL8860WT-7DICT-ND"
+			(at 0 0 180)
+			(unlocked yes)
+			(layer "F.Fab")
+			(hide yes)
+			(effects
+				(font
+					(size 1 1)
+					(thickness 0.15)
+				)
+			)
+		)
+		(property "Vendor" "DigiKey"
 			(at 0 0 180)
 			(unlocked yes)
@@
 			)
 		)
-		(property "Datasheet" ""
+		(property "Datasheet" "~"
 			(at 0 0 90)
 			(layer "F.Fab")
@@
 		)
 		(embedded_fonts no)
-		(model "C:/Users/philip.mcgaw/AppData/Local/Programs/KiCad/9.0/share/kicad/3dmodels/Connector_PinSocket_2.54mm.3dshapes/PinSocket_1x02_P2.54mm_Vertical.wrl"
+		(model "${KICAD9_3DMODEL_DIR}/Connector_PinSocket_2.54mm.3dshapes/PinSocket_1x02_P2.54mm_Vertical.wrl"
 			(offset
 				(xyz 0 0 0)
@@
 			)
 		)
-		(property "Datasheet" ""
+		(property "Datasheet" "~"
 			(at 0 0 180)
 			(layer "F.Fab")
@@
 		)
 		(embedded_fonts no)
-		(model "C:/Users/philip.mcgaw/AppData/Local/Programs/KiCad/9.0/share/kicad/3dmodels/Connector_PinSocket_2.54mm.3dshapes/PinSocket_1x02_P2.54mm_Vertical.wrl"
+		(model "${KICAD9_3DMODEL_DIR}/Connector_PinSocket_2.54mm.3dshapes/PinSocket_1x02_P2.54mm_Vertical.wrl"
 			(offset
 				(xyz 0 0 0)
@@
 			)
 		)
-		(property "Datasheet" "~"
+		(property "Datasheet" "https://www.yageo.com/upload/media/product/app/datasheet/rchip/pyu-rl_group_521_rohs_l.pdf"
 			(at 0 0 90)
 			(layer "F.Fab")
@@
 		)
 		(property "Part #" "311-0.5LWCT-ND"
+			(at 0 0 90)
+			(unlocked yes)
+			(layer "F.Fab")
+			(hide yes)
+			(effects
+				(font
+					(size 1 1)
+					(thickness 0.15)
+				)
+			)
+		)
+		(property "Vendor" "DigiKey"
 			(at 0 0 90)
 			(unlocked yes)
@@
 			)
 		)
-		(property "Datasheet" "~"
+		(property "Datasheet" "https://www.yageo.com/upload/media/product/app/datasheet/rchip/pyu-rl_group_521_rohs_l.pdf"
 			(at 0 0 90)
 			(layer "F.Fab")
@@
 		)
 		(property "Part #" "311-0.5LWCT-ND"
+			(at 0 0 90)
+			(unlocked yes)
+			(layer "F.Fab")
+			(hide yes)
+			(effects
+				(font
+					(size 1 1)
+					(thickness 0.15)
+				)
+			)
+		)
+		(property "Vendor" "DigiKey"
 			(at 0 0 90)
 			(unlocked yes)
@@
 			)
 		)
+		(property "Vendor" "DigiKey"
+			(at 0 0 0)
+			(unlocked yes)
+			(layer "B.Fab")
+			(hide yes)
+			(effects
+				(font
+					(size 1 1)
+					(thickness 0.15)
+				)
+				(justify mirror)
+			)
+		)
 		(property ki_fp_filters "LED* LED_SMD:* LED_THT:*")
 		(sheetname "/")
@@
 			)
 		)
-		(property "Datasheet" ""
+		(property "Datasheet" "~"
 			(at 0 0 0)
 			(layer "F.Fab")
@@
 		)
 		(embedded_fonts no)
-		(model "C:/Users/philip.mcgaw/AppData/Local/Programs/KiCad/9.0/share/kicad/3dmodels/Connector_PinHeader_2.54mm.3dshapes/PinHeader_1x03_P2.54mm_Vertical.wrl"
+		(model "${KICAD9_3DMODEL_DIR}/Connector_PinHeader_2.54mm.3dshapes/PinHeader_1x03_P2.54mm_Vertical.wrl"
 			(offset
 				(xyz 0 0 0)
@@
 			)
 		)
-		(property "Datasheet" ""
+		(property "Datasheet" "~"
 			(at 0 0 90)
 			(layer "F.Fab")
@@
 		)
 		(embedded_fonts no)
-		(model "C:/Users/philip.mcgaw/AppData/Local/Programs/KiCad/9.0/share/kicad/3dmodels/Connector_PinHeader_2.54mm.3dshapes/PinHeader_1x02_P2.54mm_Vertical.wrl"
+		(model "${KICAD9_3DMODEL_DIR}/Connector_PinHeader_2.54mm.3dshapes/PinHeader_1x02_P2.54mm_Vertical.wrl"
 			(offset
 				(xyz 0 0 0)
@@
 			)
 		)
-		(property "Datasheet" ""
+		(property "Datasheet" "~"
 			(at 0 0 180)
 			(layer "F.Fab")
@@
 		)
 		(embedded_fonts no)
-		(model "{{KICAD9_3DMODEL_DIR}}/3dmodels/Connector_PinHeader_2.54mm.3dshapes/PinHeader_1x02_P2.54mm_Vertical.wrl"
+		(model "${KICAD9_3DMODEL_DIR}/Connector_PinHeader_2.54mm.3dshapes/PinHeader_1x02_P2.54mm_Vertical.wrl"
 			(offset
 				(xyz 0 0 0)
@@
 	)
 	(segment
+		(start 136.16 105.2)
+		(end 135.74 105.62)
+		(width 0.5)
+		(layer "F.Cu")
+		(net 4)
+	)
+	(segment
+		(start 135.74 105.62)
+		(end 135.74 108)
+		(width 0.5)
+		(layer "F.Cu")
+		(net 4)
+	)
+	(segment
 		(start 129.256714 98.708286)
 		(end 129.976 98.708286)
@@
 	)
 	(segment
-		(start 136.16 105.2)
-		(end 136.16 107.58)
-		(width 0.5)
-		(layer "F.Cu")
-		(net 4)
-	)
-	(segment
 		(start 129.252 103.8)
 		(end 134.76 103.8)
-		(width 0.5)
-		(layer "F.Cu")
-		(net 4)
-	)
-	(segment
-		(start 136.16 107.58)
-		(end 135.74 108)
 		(width 0.5)
 		(layer "F.Cu")
@@
 			)
 		)
+	)
+	(zone
+		(net 6)
+		(net_name "/LED+{slash}U")
+		(layer "B.Cu")
+		(hatch edge 0.5)
+		(priority 2)
+		(connect_pads
+			(clearance 0.508)
+		)
+		(min_thickness 0.25)
+		(filled_areas_thickness no)
+		(fill yes
+			(thermal_gap 0.5)
+			(thermal_bridge_width 0.5)
+		)
+		(polygon
+			(pts
+				(xy 87.63 111.76) (xy 87.63 101.6) (xy 111.76 99.06) (xy 111.76 111.76)
+			)
+		)
+	)
+	(zone
+		(net 7)
+		(net_name "/LED-{slash}U")
+		(layer "B.Cu")
+		(hatch edge 0.5)
+		(priority 1)
+		(connect_pads
+			(clearance 0.508)
+		)
+		(min_thickness 0.25)
+		(filled_areas_thickness no)
+		(fill yes
+			(thermal_gap 0.5)
+			(thermal_bridge_width 0.5)
+		)
+		(polygon
+			(pts
+				(xy 87.63 88.9) (xy 111.76 88.9) (xy 111.76 97.79) (xy 87.63 100.33)
+			)
+		)

Commit message: resources
Routing:
- net /LED+/U: track 18.5 -> 0.00 mm
- net /LED-/U: track 15.9 -> 0.00 mm
Changed lines of the file:
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@@
-	)
-	(segment
-		(start 101.91 109)
-		(end 105.455 105.455)
-		(width 2)
-		(layer "B.Cu")
-		(net 6)
-	)
-	(segment
-		(start 91 109)
-		(end 101.91 109)
-		(width 2)
-		(layer "B.Cu")
-		(net 6)
-	)
-	(segment
-		(start 91 109)
-		(end 91 106.46)
-		(width 2)
-		(layer "B.Cu")
-		(net 6)
-	)
-	(segment
-		(start 109 91)
-		(end 106.46 91)
-		(width 2)
-		(layer "B.Cu")
-		(net 7)
-	)
-	(segment
-		(start 106.46 91)
-		(end 98.09 91)
-		(width 2)
-		(layer "B.Cu")
-		(net 7)
-	)
-	(segment
-		(start 98.09 91)
-		(end 94.545 94.545)
-		(width 2)
-		(layer "B.Cu")
-		(net 7)
 	)
 	(segment
@@
 		(polygon
 			(pts
-				(xy 87.63 111.76) (xy 87.63 101.6) (xy 111.76 99.06) (xy 111.76 111.76)
+				(xy 88.646 111.76) (xy 88.646 101.493053) (xy 111.2774 99.1108) (xy 111.2774 111.76)
 			)
 		)
@@
 		(polygon
 			(pts
-				(xy 87.63 88.9) (xy 111.76 88.9) (xy 111.76 97.79) (xy 87.63 100.33)
+				(xy 88.6714 88.9) (xy 111.252 88.9) (xy 111.252 98.530619) (xy 88.6714 100.907525)
 			)
 		)
