File: KiCAD/TopSide/OpenROV Topside Interface 2.6A.kicad_sch (KiCad schematic)
At the start: 20 parts, among them J1 FCI 10033526-N3212MLF, J2 FCI 20020303-D021, J3 SSW-103-01-G-D, J4 SSW-103-01-G-D, J5 HDR_1X2X0.100-ALT_SILK, U1 AP1117IE33G

Commit message: change
Other:
- note removed: "11 Feb 2014"
- note removed: "2.6"
- note removed: "2.6A"
- note removed: "26 Nov 2013"
- note removed: "Changes"
- note removed: "Date"
- note removed: "Engr"
- note removed: "Initial Prototype"
- note removed: "No schematic changes from Rev 2.6. Positions of J1 and J2 adjusted. Longer engagement length on headers J3 and J4. Revised silkscreen and soldermask. Hole for optional standoff."
- note removed: "RWH"
- note removed: "Rev"
- note removed: "Revision History"
